Commit message: adding camera

File: description/camera.xacro (robot description, xacro)
@@ -1,6 +1,3 @@
 <?xml version="1.0"?>
-<<<<<<< HEAD
-<robot>
-=======
 <robot>
     <joint name="camera_joint" type="fixed">
@@ -15,5 +12,4 @@
     </joint>
     <link name="camera_link_optical"></link>
->>>>>>> 7a61ef2b9ed9047d0898131a1162ec252a2a4513
     <link name="camera_link">
         <visual>
@@ -24,23 +20,6 @@
         </visual>
     </link>
-<<<<<<< HEAD
-    <joint name="camera_joint" type="fixed">
-        <parent link="chassis"/>
-        <child link="camera_link"/>
-        <origin xyz="0.305 0 0.08" rpy="0.0 0.0 0.0"/>
-    </joint>
-    <joint name="camera_optical_joint" type="fixed">
-        <parent link="camera_link"/>
-        <child link="camera_link_optical"/>
-        <origin xyz="0 0 0" rpy="${-pi/2} 0 ${-pi/2}"/>
-    </joint>
-    <link name="camera_link_optical"></link>
     <gazebo reference="camera_link">
         <material>Gazebo/Red</material>
     </gazebo>
-=======
-    <gazebo reference="camera_link">
-        <material>Gazebo/Red</material>
-    </gazebo>
->>>>>>> 7a61ef2b9ed9047d0898131a1162ec252a2a4513
 </robot>

Commit message: test lidar

File: description/camera.xacro (robot description, xacro)
@@ -1,4 +1,4 @@
 <?xml version="1.0"?>
-<robot>
+<robot xmlns:xacro="http://www.ros.org/wiki/xacro" xmlns:gz="http://gazebosim.org/xmlschema/gz/1.0" name="camera">
     <joint name="camera_joint" type="fixed">
         <parent link="chassis"/>

File: description/lidar.xacro (robot description, xacro)
@@ -4,5 +4,5 @@
         <parent link="chassis"/>
         <child link="laser_frame"/>
-        <origin xyz="0.1 0 0.175" rpy="0 0 0"/>
+        <origin xyz="0.122 0 0.212" rpy="0 0 0"/>
     </joint>
     <link name="laser_frame">
@@ -12,4 +12,11 @@
             </geometry>
             <material name="red"/>
+        </visual>
+        <visual>
+            <origin xyz="0 0 -0.05"/>
+            <geometry>
+                <cylinder radius="0.01" length="0.1"/>
+            </geometry>
+            <material name="black"/>
         </visual>
         <collision>
@@ -23,8 +30,8 @@
     </link>
     <gazebo reference="laser_frame">
-        <material>Gazebo/Red</material>
+        <material>Gazebo/Black</material>
         <sensor name="laser" type="gpu_lidar">
             <pose> 0 0 0 0 0 0 </pose>
-            <visualize>true</visualize>
+            <visualize>false</visualize>
             <update_rate>10</update_rate>
             <lidar>
@@ -32,5 +39,4 @@
                     <horizontal>
                         <samples>360</samples>
-                        <resolution>1</resolution>
                         <min_angle>-3.14</min_angle>
                         <max_angle>3.14</max_angle>
@@ -40,5 +46,4 @@
                     <min>0.3</min>
                     <max>12</max>
-                    <resolution>0.01</resolution>
                 </range>
             </lidar>

Commit message: Jason TODO #1 done

File: description/camera.xacro (robot description, xacro)
@@ -1,15 +1,9 @@
 <?xml version="1.0"?>
-<robot xmlns:xacro="http://www.ros.org/wiki/xacro" xmlns:gz="http://gazebosim.org/xmlschema/gz/1.0" name="camera">
+<robot xmlns:xacro="http://www.ros.org/wiki/xacro">
     <joint name="camera_joint" type="fixed">
         <parent link="chassis"/>
         <child link="camera_link"/>
-        <origin xyz="0.305 0.0 0.08" rpy="0.0 0.0 0.0"/>
+        <origin xyz="0.276 0.0 0.08" rpy="0.0 0.18 0.0"/>
     </joint>
-    <joint name="camera_optical_joint" type="fixed">
-        <parent link="camera_link"/>
-        <child link="camera_link_optical"/>
-        <origin xyz="0.0 0.0 0.0" rpy="${-pi/2} 0 ${-pi/2}"/>
-    </joint>
-    <link name="camera_link_optical"></link>
     <link name="camera_link">
         <visual>
@@ -19,5 +13,18 @@
             <material name="red"/>
         </visual>
+        <visual>
+            <origin xyz="0 0 -0.05"/>
+            <geometry>
+                <cylinder radius="0.002" length="0.1"/>
+            </geometry>
+            <material name="blue"/>
+        </visual>
     </link>
+    <joint name="camera_optical_joint" type="fixed">
+        <parent link="camera_link"/>
+        <child link="camera_link_optical"/>
+        <origin xyz="0.0 0.0 0.0" rpy="${-pi/2} 0 ${-pi/2}"/>
+    </joint>
+    <link name="camera_link_optical"></link>
     <gazebo reference="camera_link">
         <material>Gazebo/Red</material>

Commit message: more stuff

File: description/camera.xacro (robot description, xacro)
@@ -4,5 +4,5 @@
         <parent link="chassis"/>
         <child link="camera_link"/>
-        <origin xyz="0.276 0.0 0.08" rpy="0.0 0.18 0.0"/>
+        <origin xyz="0.308 0.0 0.08" rpy="0.0 0.18 0.0"/>
     </joint>
     <link name="camera_link">

File: description/lidar.xacro (robot description, xacro)
@@ -35,5 +35,5 @@
             <visualize>true</visualize>
             <update_rate>10</update_rate>
-            <ray>
+            <lidar>
                 <scan>
                     <horizontal>
@@ -47,5 +47,5 @@
                     <max>12</max>
                 </range>
-            </ray>
+            </lidar>
             <topic>lidar</topic>
             <gz_frame_id>laser_frame</gz_frame_id>

File: description/robot.urdf.xacro (robot description, xacro)
@@ -36,5 +36,5 @@
                 <box size="0.3 0.3 0.15"/>
             </geometry>
-            <material name="white"></material>
+            <material name="black"></material>
         </visual>
    </link>
