Commit message: rebuilt to add left wheel/link

File: description/robot.urdf.xacro (robot description, xacro)
@@ -1,15 +1,19 @@
 <?xml version="1.0"?>
 <robot xmlns:xacro="http://www.ros.org/wiki/xacro"  name="robot">
+<xacro:include filename="inertial_macros.xacro" />
     <material name="white">
-        <color rgba="1 1 1 1"/>
+        <color rgba="1 1 1 1" />
+    </material>
+    <material name="black">
+        <color rgba="0 0 0 1" />
     </material>
     <material name="orange">
-        <color rgba="1 0.3 0.1 1"/>
+        <color rgba="1 0.3 0.1 1" />
     </material>
     <material name="blue">
-        <color rgba="0.2 0.2 1 1"/>
+        <color rgba="0.2 0.2 1 1" />
     </material>
-    <material name="black">
-        <color rgba="0 0 0 1"/>
+    <material name="green">
+        <color rgba="0 0.3 0 1" />
     </material>
     <!-- Example link -->
@@ -29,3 +33,25 @@
         </visual>
    </link>
+    <joint name="left_wheel_joint" type="continuous">
+        <parent link="base_link" />
+        <child link="left_wheel" />
+        <origin xyz="0.0 0.175 0.0" rpy="-${pi/2} 0.0 0.0" />
+        <axis xyz="0.0 0.0 1.0" />
+    </joint>
+    <link name="left_wheel">
+        <visual>
+            <geometry>
+                <cylinder radius="0.04" length="0.05" />
+            </geometry>
+            <material name="green" />
+        </visual>
+        <collision>
+            <geometry>
+                <cylinder radius="0.04" length="0.05" />
+            </geometry>
+        </collision>
+        <xacro:inertial_cylinder mass="0.1" radius="0.04" length="0.05">
+            <origin xyz="0.0 0.0 0.0" rpy="0.0 0.0 0.0" />
+        </xacro:inertial_cylinder>
+    </link>
 </robot>

Commit message: rebuilt to add right wheel; moved files to dev_ws

File: description/robot.urdf.xacro (robot description, xacro)
@@ -55,3 +55,25 @@
         </xacro:inertial_cylinder>
     </link>
+    <joint name="right_wheel_joint" type="continuous">
+        <parent link="base_link" />
+        <child link="right_wheel" />
+        <origin xyz="0.0 -0.175 0.0" rpy="${pi/2} 0.0 0.0" />
+        <axis xyz="0.0 0.0 1.0" />
+    </joint>
+    <link name="right_wheel">
+        <visual>
+            <geometry>
+                <cylinder radius="0.04" length="0.05" />
+            </geometry>
+            <material name="green" />
+        </visual>
+        <collision>
+            <geometry>
+                <cylinder radius="0.04" length="0.05" />
+            </geometry>
+        </collision>
+        <xacro:inertial_cylinder mass="0.1" radius="0.04" length="0.05">
+            <origin xyz="0.0 0.0 0.0" rpy="0.0 0.0 0.0" />
+        </xacro:inertial_cylinder>
+    </link>
 </robot>

Commit message: added caster wheel

File: description/robot.urdf.xacro (robot description, xacro)
@@ -77,3 +77,19 @@
         </xacro:inertial_cylinder>
     </link>
+    <link name="caster_wheel">
+        <visual>
+            <geometry>
+                <sphere radius="0.05"/>
+            </geometry>
+            <material name="black"/>
+        </visual>
+        <collision>
+            <geometry>
+                <sphere radius="0.05"/>
+            </geometry>
+        </collision>
+        <xacro:inertial_sphere mass="0.1" radius="0.05">
+            <origin xyz="0 0 0" rpy="0 0 0"/>
+        </xacro:inertial_sphere>
+    </link>
 </robot>

Commit message: added caster joint bc forgot

File: description/robot.urdf.xacro (robot description, xacro)
@@ -77,4 +77,9 @@
         </xacro:inertial_cylinder>
     </link>
+    <joint name="caster_wheel_joint" type="fixed">
+        <parent link="chassis"/>
+        <child link="caster_wheel"/>
+        <origin xyz="0.24 0 0"/>
+    </joint>
     <link name="caster_wheel">
         <visual>

Commit message: gazebo control plugin issue

File: description/robot.urdf.xacro (robot description, xacro)
@@ -2,4 +2,5 @@
 <robot xmlns:xacro="http://www.ros.org/wiki/xacro"  name="robot">
 <xacro:include filename="inertial_macros.xacro" />
+<xacro:include filename="gazebo_control.xacro" />
     <material name="white">
         <color rgba="1 1 1 1" />
@@ -30,7 +31,10 @@
                 <box size="0.3 0.3 0.15"/>
             </geometry>
-            <material name="black"></material>
+            <material name="white"></material>
         </visual>
    </link>
+   <gazebo reference="chassis">
+    <material>Gazebo/White</material>
+   </gazebo>
     <joint name="left_wheel_joint" type="continuous">
         <parent link="base_link" />
@@ -44,5 +48,5 @@
                 <cylinder radius="0.04" length="0.05" />
             </geometry>
-            <material name="green" />
+            <material name="blue" />
         </visual>
         <collision>
@@ -55,4 +59,7 @@
         </xacro:inertial_cylinder>
     </link>
+    <gazebo reference="left_wheel">
+        <material>Gazebo/Blue</material>
+   </gazebo>
     <joint name="right_wheel_joint" type="continuous">
         <parent link="base_link" />
@@ -66,5 +73,5 @@
                 <cylinder radius="0.04" length="0.05" />
             </geometry>
-            <material name="green" />
+            <material name="blue" />
         </visual>
         <collision>
@@ -77,4 +84,7 @@
         </xacro:inertial_cylinder>
     </link>
+    <gazebo reference="right_wheel">
+        <material>Gazebo/Blue</material>
+   </gazebo>
     <joint name="caster_wheel_joint" type="fixed">
         <parent link="chassis"/>
@@ -98,3 +108,6 @@
         </xacro:inertial_sphere>
     </link>
+    <gazebo reference="caster_wheel">
+        <material>Gazebo/Black</material>
+   </gazebo>
 </robot>

Commit message: changed back the robot color to original

File: description/robot.urdf.xacro (robot description, xacro)
@@ -31,9 +31,9 @@
                 <box size="0.3 0.3 0.15"/>
             </geometry>
-            <material name="white"></material>
+            <material name="black"></material>
         </visual>
    </link>
    <gazebo reference="chassis">
-    <material>Gazebo/White</material>
+    <material>Gazebo/Black</material>
    </gazebo>
     <joint name="left_wheel_joint" type="continuous">
@@ -48,5 +48,5 @@
                 <cylinder radius="0.04" length="0.05" />
             </geometry>
-            <material name="blue" />
+            <material name="green" />
         </visual>
         <collision>
@@ -60,5 +60,5 @@
     </link>
     <gazebo reference="left_wheel">
-        <material>Gazebo/Blue</material>
+        <material>Gazebo/Green</material>
    </gazebo>
     <joint name="right_wheel_joint" type="continuous">
@@ -73,5 +73,5 @@
                 <cylinder radius="0.04" length="0.05" />
             </geometry>
-            <material name="blue" />
+            <material name="green" />
         </visual>
         <collision>
@@ -85,5 +85,5 @@
     </link>
     <gazebo reference="right_wheel">
-        <material>Gazebo/Blue</material>
+        <material>Gazebo/Green</material>
    </gazebo>
     <joint name="caster_wheel_joint" type="fixed">
@@ -97,5 +97,5 @@
                 <sphere radius="0.05"/>
             </geometry>
-            <material name="black"/>
+            <material name="white"/>
         </visual>
         <collision>
@@ -109,5 +109,5 @@
     </link>
     <gazebo reference="caster_wheel">
-        <material>Gazebo/Black</material>
+        <material>Gazebo/White</material>
    </gazebo>
 </robot>

Commit message: Add ros2_control to gazebo

File: description/robot.urdf.xacro (robot description, xacro)
@@ -1,7 +1,8 @@
 <?xml version="1.0"?>
-<robot xmlns:xacro="http://www.ros.org/wiki/xacro"  name="robot">
-<xacro:include filename="inertial_macros.xacro" />
-<xacro:include filename="gazebo_control.xacro" />
-<xacro:include filename="camera.xacro" />
+<robot xmlns:xacro="http://www.ros.org/wiki/xacro" name="robot">
+    <xacro:include filename="inertial_macros.xacro" />
+    <!-- <xacro:include filename="gazebo_control.xacro" /> -->
+    <xacro:include filename="ros2_control.xacro" />
+    <xacro:include filename="camera.xacro" />
     <material name="white">
         <color rgba="1 1 1 1" />
@@ -21,21 +22,21 @@
     <!-- Example link -->
     <link name="base_link"></link>
-   <joint name="chassis_joint" type="fixed">
-    <parent link="base_link"/>
-    <child link="chassis"/>
-    <origin xyz="-0.1 0.0 0.0" rpy="0.0 0.0 0.0"/>
-   </joint>
-   <link name="chassis">
+    <joint name="chassis_joint" type="fixed">
+        <parent link="base_link" />
+        <child link="chassis" />
+        <origin xyz="-0.1 0.0 0.0" rpy="0.0 0.0 0.0" />
+    </joint>
+    <link name="chassis">
         <visual>
-            <origin xyz="0.15 0.0 0.075" rpy="0.0 0.0 0.0"/>
+            <origin xyz="0.15 0.0 0.075" rpy="0.0 0.0 0.0" />
             <geometry>
-                <box size="0.3 0.3 0.15"/>
+                <box size="0.3 0.3 0.15" />
             </geometry>
             <material name="black"></material>
         </visual>
-   </link>
-   <gazebo reference="chassis">
-    <material>Gazebo/Black</material>
-   </gazebo>
+    </link>
+    <gazebo reference="chassis">
+        <material>Gazebo/Black</material>
+    </gazebo>
     <joint name="left_wheel_joint" type="continuous">
         <parent link="base_link" />
@@ -62,5 +63,5 @@
     <gazebo reference="left_wheel">
         <material>Gazebo/Green</material>
-   </gazebo>
+    </gazebo>
     <joint name="right_wheel_joint" type="continuous">
         <parent link="base_link" />
@@ -87,28 +88,28 @@
     <gazebo reference="right_wheel">
         <material>Gazebo/Green</material>
-   </gazebo>
+    </gazebo>
     <joint name="caster_wheel_joint" type="fixed">
-        <parent link="chassis"/>
-        <child link="caster_wheel"/>
-        <origin xyz="0.24 0 0"/>
+        <parent link="chassis" />
+        <child link="caster_wheel" />
+        <origin xyz="0.24 0 0" />
     </joint>
     <link name="caster_wheel">
         <visual>
             <geometry>
-                <sphere radius="0.05"/>
+                <sphere radius="0.05" />
             </geometry>
-            <material name="white"/>
+            <material name="white" />
         </visual>
         <collision>
             <geometry>
-                <sphere radius="0.05"/>
+                <sphere radius="0.05" />
             </geometry>
         </collision>
         <xacro:inertial_sphere mass="0.1" radius="0.05">
-            <origin xyz="0 0 0" rpy="0 0 0"/>
+            <origin xyz="0 0 0" rpy="0 0 0" />
         </xacro:inertial_sphere>
     </link>
     <gazebo reference="caster_wheel">
         <material>Gazebo/White</material>
-   </gazebo>
+    </gazebo>
 </robot>

Commit message: added LiDar and Camera, Ye Chan test since Jason's PC cannot show the rays and camera frame

File: description/robot.urdf.xacro (robot description, xacro)
@@ -4,4 +4,5 @@
 <xacro:include filename="gazebo_control.xacro" />
 <xacro:include filename="camera.xacro" />
+<xacro:include filename="lidar.xacro" />
     <material name="white">
         <color rgba="1 1 1 1" />
@@ -19,4 +20,7 @@
         <color rgba="0 0.3 0 1" />
     </material>
+    <material name="red">
+        <color rgba="1 0 0 1" />
+    </material>
     <!-- Example link -->
     <link name="base_link"></link>
@@ -32,5 +36,5 @@
                 <box size="0.3 0.3 0.15"/>
             </geometry>
-            <material name="black"></material>
+            <material name="white"></material>
         </visual>
    </link>

Commit message: rviz update -> finally worke

File: description/robot.urdf.xacro (robot description, xacro)
@@ -42,10 +42,4 @@
     <material>Gazebo/Black</material>
    </gazebo>
-    <joint name="left_wheel_joint" type="continuous">
-        <parent link="base_link" />
-        <child link="left_wheel" />
-        <origin xyz="0.0 0.175 0.0" rpy="-${pi/2} 0.0 0.0" />
-        <axis xyz="0.0 0.0 1.0" />
-    </joint>
     <link name="left_wheel">
         <visual>
@@ -64,13 +58,13 @@
         </xacro:inertial_cylinder>
     </link>
+    <joint name="left_wheel_joint" type="continuous">
+        <parent link="base_link" />
+        <child link="left_wheel" />
+        <origin xyz="0.0 0.175 0.0" rpy="-${pi/2} 0.0 0.0" />
+        <axis xyz="0.0 0.0 1.0" />
+    </joint>
     <gazebo reference="left_wheel">
         <material>Gazebo/Green</material>
    </gazebo>
-    <joint name="right_wheel_joint" type="continuous">
-        <parent link="base_link" />
-        <child link="right_wheel" />
-        <origin xyz="0.0 -0.175 0.0" rpy="${pi/2} 0.0 0.0" />
-        <axis xyz="0.0 0.0 1.0" />
-    </joint>
     <link name="right_wheel">
         <visual>
@@ -89,4 +83,10 @@
         </xacro:inertial_cylinder>
     </link>
+    <joint name="right_wheel_joint" type="continuous">
+        <parent link="base_link" />
+        <child link="right_wheel" />
+        <origin xyz="0.0 -0.175 0.0" rpy="${pi/2} 0.0 0.0" />
+        <axis xyz="0.0 0.0 1.0" />
+    </joint>
     <gazebo reference="right_wheel">
         <material>Gazebo/Green</material>
